File: hardware/starbie_pet/starbie_pet.kicad_sch (KiCad schematic)
At the start: 15 parts, among them J1 DHT11, J2 LiPo, J3 Conn_01x04_Socket, J4 ST7789_(display), J6 MPU6050, J7 espleft, J8 espright, J9 Out1, SW1 SW_Push, SW2 SW_Push, SW3 SW_SPST

Commit message: Add PCB files
Parts:
- removed J1: DHT11, symbol Connector:Conn_01x03_Socket
- removed J2: LiPo, Sensor_Motion:InvenSense_QFN-24_4x4mm_P0.5mm, symbol Connector_Generic:Conn_01x02
- removed J3: Conn_01x04_Socket, symbol Connector:Conn_01x04_Socket
- removed J4: ST7789_(display), Sensor_Motion:InvenSense_QFN-24_4x4mm_P0.5mm, symbol Connector_Generic:Conn_01x08
- removed J6: MPU6050, symbol Connector_Generic:Conn_01x08
- removed J7: espleft, symbol Connector:Conn_01x15_Socket
- removed J8: espright, symbol Connector:Conn_01x15_Socket
- removed J9: Out1, symbol Connector:Conn_01x02_Socket
- removed SW3: SW_SPST, Button_Switch_THT:SW_NKK_GW12LJP, symbol Switch:SW_SPST
- added DHT11temp1: Conn_01x03_Socket, Connector_PinSocket_2.54mm:PinSocket_1x03_P2.54mm_Vertical, symbol Connector:Conn_01x03_Socket
- added GyroMPU6050, display1: Conn_01x08_Socket, Connector_PinSocket_2.54mm:PinSocket_1x08_P2.54mm_Vertical, symbol Connector:Conn_01x08_Socket
- added H1, H2, H3, H4: MountingHole, MountingHole:MountingHole_3.2mm_M3, symbol Mechanical:MountingHole
- added Out1: Conn_01x02_Socket, Connector_PinHeader_2.54mm:PinHeader_1x02_P2.54mm_Vertical, symbol Connector:Conn_01x02_Socket
- added Powerswitch1: SW_SPST, Connector:FanPinHeader_1x03_P2.54mm_Vertical, symbol Switch:SW_SPST
- added battery2: Conn_01x02_Socket, Connector_JST:JST_PH_B2B-PH-K_1x02_P2.00mm_Vertical, symbol Connector:Conn_01x02_Socket
- added charging1: Conn_01x04_Socket, Connector:FanPinHeader_1x04_P2.54mm_Vertical, symbol Connector:Conn_01x04_Socket
- added espleft1, espright1: Conn_01x15_Socket, Connector_PinSocket_2.54mm:PinSocket_1x15_P2.54mm_Vertical, symbol Connector:Conn_01x15_Socket
- Input1: footprint (none) -> Connector_PinHeader_2.54mm:PinHeader_1x02_P2.54mm_Vertical
- R1batlvl1, R2batlvl1: footprint (none) -> Resistor_THT:R_Axial_DIN0207_L6.3mm_D2.5mm_P2.54mm_Vertical
- SW1: footprint Button_Switch_THT:SW_NKK_GW12LJP -> Button_Switch_THT:SW_PUSH_6mm
- SW2: footprint (none) -> Button_Switch_THT:SW_PUSH_6mm
- touchpad1: footprint (none) -> TestPoint:TestPoint_Pad_D4.0mm
Connections:
- net BUTTON2 is gone; now on net GND: SW2.2
- net +3V3: now also DHT11temp1.1 (Pin_1), GyroMPU6050.1 (Pin_1), display1.1 (Pin_1), display1.8 (Pin_8), espright1.1 (Pin_1)
- net +5V: now also Out1.1 (Pin_1), espleft1.15 (Pin_15)
- net BUTTON: now also SW1.1, espleft1.6 (Pin_6); no longer SW1.2
- net Bat_sense: now also R1batlvl1.2, R2batlvl1.1, espleft1.5 (Pin_5); no longer R1batlvl1.1, R2batlvl1.2
- net CHG_OUT: now also Powerswitch1.1 (A), charging1.1 (Pin_1)
- net DHT_DATA: now also DHT11temp1.3 (Pin_3), espright1.7 (Pin_7)
- net GND: now also R2batlvl1.2, SW1.2, DHT11temp1.2 (Pin_2), GyroMPU6050.2 (Pin_2), Out1.2 (Pin_2), charging1.4 (Pin_4), display1.7 (Pin_7), espleft1.14 (Pin_14), espright1.2 (Pin_2); no longer R2batlvl1.1, SW1.1, SW2.1
- net SPI_CLK: now also display1.2 (Pin_2), espright1.9 (Pin_9)
- net SPI_MOSI: now also display1.3 (Pin_3), espright1.15 (Pin_15)
- net TFT_CS: now also display1.6 (Pin_6), espright1.8 (Pin_8)
- net TFT_DC: now also display1.4 (Pin_4), espleft1.10 (Pin_10)
- net TFT_RST: now also display1.5 (Pin_5), espright1.5 (Pin_5)
- net TOUCH: now also espleft1.11 (Pin_11)
- net Vbat: now also R1batlvl1.1, Powerswitch1.2 (B); no longer R1batlvl1.2
- new net Bat_neg: battery2.2 (Pin_2), charging1.3 (Pin_3)
- new net Bat_pos: battery2.1 (Pin_1), charging1.2 (Pin_2)
- new net Button2: SW2.1, espright1.3 (Pin_3)
- new net EN: espleft1.1 (Pin_1)
- new net GPIO12: espleft1.12 (Pin_12)
- new net GPIO2: espright1.4 (Pin_4)
- new net GPIO34: espleft1.4 (Pin_4)
- new net GPIO36: espleft1.2 (Pin_2)
- new net GPIO39: espleft1.3 (Pin_3)
- new net I2C_SCL: GyroMPU6050.3 (Pin_3), espright1.14 (Pin_14)
- new net I2C_SDA: GyroMPU6050.4 (Pin_4), espright1.11 (Pin_11)
- new net I2S_BCLK: espleft1.9 (Pin_9)
- new net I2S_DIN: espleft1.7 (Pin_7)
- new net I2S_LRC: espleft1.8 (Pin_8)
- new net MOTOR: espright1.6 (Pin_6)
- new net RX0: espright1.12 (Pin_12)
- new net SD_CS: espleft1.13 (Pin_13)
- new net SPI_MISO: espright1.10 (Pin_10)
- new net TX0: espright1.13 (Pin_13)
Other:
- note added: "Boostconverter mt3608"

Commit message: Update schematic
Parts:
- removed H1, H2, H3, H4: MountingHole, MountingHole:MountingHole_3.2mm_M3, symbol Mechanical:MountingHole
